File: stm32.kicad_pcb (KiCad board)
At the start: 2 copper layers, 44.4 x 32.7 mm, 38 parts, among them J1 USB C Connector, J2 Conn_01x04_Male, J3 SWD_10, J4 Conn_01x04_Male, J5 Conn_01x05_Female, SW1 SW_SPDT, U1 AMS1117-3.3, U2 STM32F103C8T6, Y1 16MHz

Commit message: update infos
Changed lines of the file:
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@@
     (effects (font (size 1.2 1.2) (thickness 0.2)))
   )
-  (gr_text "JLCJLCJLCJLC" (at 79.2 87.9 45) (layer "F.SilkS")
+  (gr_text "JLCJLCJLCJLC" (at 97.3 87 90) (layer "F.SilkS")
     (effects (font (size 0.7 0.7) (thickness 0.15)))
   )
@@
     (polygon
       (pts
-        (xy 90.55 90.75)
-        (xy 90.55 93.45)
-        (xy 91 94)
-        (xy 92.95 94)
-        (xy 93.2 94.35)
-        (xy 93.2 96.05)
-        (xy 92.9 96.3)
-        (xy 91.05 96.3)
-        (xy 90.9 96)
-        (xy 89.2 96)
-        (xy 88.95 95.65)
-        (xy 88.95 92.3)
-        (xy 87.85 92.3)
-        (xy 87.6 92.05)
-        (xy 87.6 90.55)
-        (xy 87.95 90.35)
-        (xy 90.05 90.35)
+        (xy 90.65 90.75)
+        (xy 90.65 93.45)
+        (xy 91 93.95)
+        (xy 92.95 93.95)
+        (xy 93.25 94.35)
+        (xy 93.25 96.05)
+        (xy 93 96.4)
+        (xy 91.05 96.4)
+        (xy 90.9 96.1)
+        (xy 89.15 96.1)
+        (xy 88.75 95.7)
+        (xy 88.75 92.8)
+        (xy 88.6 92.4)
+        (xy 87.85 92.4)
+        (xy 87.5 92.05)
+        (xy 87.5 90.55)
+        (xy 87.95 90.3)
+        (xy 90.05 90.3)
       )
     )
@@
     (polygon
       (pts
-        (xy 88.4 92.9)
-        (xy 88.4 96.15)
-        (xy 89.15 96.75)
-        (xy 93.05 96.75)
-        (xy 93.3 97.1)
-        (xy 93.3 98.105664)
-        (xy 93.3 100.2)
-        (xy 92.65 101.2)
-        (xy 90.35 101.2)
-        (xy 89.65 101.2)
-        (xy 89.3 101.2)
-        (xy 85.5 101.2)
-        (xy 85.3 100.95)
-        (xy 85.3 97.05)
-        (xy 86.5 95.75)
-        (xy 86.5 93.151162)
-        (xy 86.5 92.8)
-        (xy 86.7 92.6)
-        (xy 88.3 92.6)
+        (xy 88.55 92.9)
+        (xy 88.55 96.2)
+        (xy 89.15 96.65)
+        (xy 93.05 96.65)
+        (xy 93.45 97.1)
+        (xy 93.45 98.1)
+        (xy 93.45 100.2)
+        (xy 92.65 101.3)
+        (xy 90.4 101.3)
+        (xy 89.7 101.3)
+        (xy 89.3 101.3)
+        (xy 85.25 101.3)
+        (xy 85 100.9)
+        (xy 85 96.95)
+        (xy 86.35 95.75)
+        (xy 86.35 93.151162)
+        (xy 86.35 92.8)
+        (xy 86.55 92.55)
+        (xy 88.4 92.55)
       )
     )
@@
         (xy 95.1 89.75)
         (xy 87.75 89.75)
-        (xy 87.15 90.35)
-        (xy 87.15 91.95)
+        (xy 87.3 90.35)
+        (xy 87.3 91.95)
         (xy 86.9 92.3)
         (xy 86.35 92.3)
