File: stm32.kicad_sch (KiCad schematic)
At the start: 37 parts, among them J1 USB C Connector, J2 Conn_01x04_Male, J3 SWD_10, J4 Conn_01x04_Male, J5 Conn_01x05_Female, SW1 SW_SPDT, U1 AMS1117-3.3, U2 STM32F103C8T6, Y1 16MHz

Commit message: update infos
Parts:
- D2: value RED -> WHITE
Changed lines of the file:
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@@
+    (pin "1")
+  )
+  (symbol (lib_id "power:VBUS") (at 228.6 106.68 0) (unit 1)
+    (in_bom yes) (on_board yes) (fields_autoplaced)
+    (property "Reference" "#PWR?" (id 0) (at 228.6 110.49 0)
+      (effects (font (size 1.27 1.27)) hide)
+    )
+    (property "Value" "VBUS" (id 1) (at 228.6 101.6 0))
+    (property "Footprint" "" (id 2) (at 228.6 106.68 0)
+      (effects (font (size 1.27 1.27)) hide)
+    )
+    (property "Datasheet" "" (id 3) (at 228.6 106.68 0)
+      (effects (font (size 1.27 1.27)) hide)
+    )
     (pin "1")
   )
@@
     (pin "1")
     (pin "2")
-  )
-  (symbol (lib_id "power:VBUS") (at 237.49 106.68 0) (unit 1)
-    (in_bom yes) (on_board yes) (fields_autoplaced)
-    (property "Reference" "#PWR013" (id 0) (at 237.49 110.49 0)
-      (effects (font (size 1.27 1.27)) hide)
-    )
-    (property "Value" "VBUS" (id 1) (at 237.49 101.6 0))
-    (property "Footprint" "" (id 2) (at 237.49 106.68 0)
-      (effects (font (size 1.27 1.27)) hide)
-    )
-    (property "Datasheet" "" (id 3) (at 237.49 106.68 0)
-      (effects (font (size 1.27 1.27)) hide)
-    )
-    (pin "1")
   )
   (symbol (lib_id "Device:Crystal_GND24") (at 92.71 88.9 0) (unit 1)
@@
     (pin "2")
     (pin "3")
+  )
+  (symbol (lib_id "power:PWR_FLAG") (at 237.49 106.68 0) (unit 1)
+    (in_bom yes) (on_board yes) (fields_autoplaced)
+    (property "Reference" "#FLG?" (id 0) (at 237.49 104.775 0)
+      (effects (font (size 1.27 1.27)) hide)
+    )
+    (property "Value" "PWR_FLAG" (id 1) (at 237.49 101.6 0))
+    (property "Footprint" "" (id 2) (at 237.49 106.68 0)
+      (effects (font (size 1.27 1.27)) hide)
+    )
+    (property "Datasheet" "~" (id 3) (at 237.49 106.68 0)
+      (effects (font (size 1.27 1.27)) hide)
+    )
+    (pin "1")
   )
   (symbol (lib_id "MCU_ST_STM32F1:STM32F103C8Tx") (at 137.16 104.14 0) (unit 1)
@@
     (pin "1")
   )
-  (symbol (lib_id "power:PWR_FLAG") (at 228.6 106.68 0) (unit 1)
-    (in_bom yes) (on_board yes) (fields_autoplaced)
-    (property "Reference" "#FLG0102" (id 0) (at 228.6 104.775 0)
-      (effects (font (size 1.27 1.27)) hide)
-    )
-    (property "Value" "PWR_FLAG" (id 1) (at 228.6 101.6 0))
-    (property "Footprint" "" (id 2) (at 228.6 106.68 0)
-      (effects (font (size 1.27 1.27)) hide)
-    )
-    (property "Datasheet" "~" (id 3) (at 228.6 106.68 0)
-      (effects (font (size 1.27 1.27)) hide)
-    )
-    (pin "1")
-  )
   (symbol (lib_id "Mechanical:MountingHole") (at 25.4 115.57 0) (unit 1)
     (in_bom yes) (on_board yes) (fields_autoplaced)
@@
     (in_bom yes) (on_board yes)
     (property "Reference" "D2" (id 0) (at 140.97 168.91 0))
-    (property "Value" "RED" (id 1) (at 140.97 171.45 0))
+    (property "Value" "WHITE" (id 1) (at 140.97 171.45 0))
     (property "Footprint" "LED_SMD:LED_0603_1608Metric" (id 2) (at 140.97 173.99 0)
       (effects (font (size 1.27 1.27)) hide)
@@
       (reference "#FLG0101") (unit 1) (value "PWR_FLAG") (footprint "")
     )
-    (path "/7a4dd703-14bc-4cf8-bc14-86c2b20a5782"
-      (reference "#FLG0102") (unit 1) (value "PWR_FLAG") (footprint "")
+    (path "/69a7c179-446b-4bd9-a02d-6edec9d9c191"
+      (reference "#FLG?") (unit 1) (value "PWR_FLAG") (footprint "")
     )
     (path "/72ec0f5d-975b-472f-83a2-07c9869e6177"
@@
       (reference "#PWR012") (unit 1) (value "GND") (footprint "")
     )
-    (path "/198c41fc-1322-4478-b85f-35c279148562"
-      (reference "#PWR013") (unit 1) (value "VBUS") (footprint "")
-    )
     (path "/128c1301-b8f5-4f3a-aff5-31e07ca165ec"
       (reference "#PWR014") (unit 1) (value "GND") (footprint "")
@@
       (reference "#PWR0102") (unit 1) (value "GND") (footprint "")
     )
+    (path "/06c05959-0355-4e5e-b5fd-d3a70203028b"
+      (reference "#PWR?") (unit 1) (value "VBUS") (footprint "")
+    )
     (path "/7e23f363-4338-4760-bfd5-59d2a11ccf99"
       (reference "C1") (unit 1) (value "22u") (footprint "Capacitor_SMD:C_0805_2012Metric")
@@
     )
     (path "/ce665a87-e4e3-4201-9123-d7f12a0de959"
-      (reference "D2") (unit 1) (value "RED") (footprint "LED_SMD:LED_0603_1608Metric")
+      (reference "D2") (unit 1) (value "WHITE") (footprint "LED_SMD:LED_0603_1608Metric")
     )
     (path "/cabae09a-cd34-4fc3-9711-77ba614aac6c"
